File: Esquematicos/modulo 4/lipo.sch (KiCad schematic (older format))
At the start: 8 parts

Commit message: cambios
Parts:
- gave numbers to parts that had none: 8
Changed lines of the file:
@@
 Sheet 3 3
 Title ""
-Date "18 feb 2014"
+Date "19 feb 2014"
 Rev ""
 Comp ""
@@
 $EndDescr
 $Comp
-L BQ24210 U?
+L BQ24210 U5
 U 1 1 5302A303
 P 5750 4200
-F 0 "U?" H 5750 3750 60  0000 C CNN
+F 0 "U5" H 5750 3750 60  0000 C CNN
 F 1 "BQ24210" H 5780 4650 60  0000 C CNN
 F 2 "~" H 5800 4100 60  0000 C CNN
@@
 $EndComp
 $Comp
-L +5V #PWR?
+L +5V #PWR021
 U 1 1 5302A312
 P 5000 3800
-F 0 "#PWR?" H 5000 3890 20  0001 C CNN
+F 0 "#PWR021" H 5000 3890 20  0001 C CNN
 F 1 "+5V" H 5000 3890 30  0000 C CNN
 F 2 "" H 5000 3800 60  0000 C CNN
@@
 $EndComp
 $Comp
-L C C?
+L C C10
 U 1 1 5302A322
 P 4000 4150
-F 0 "C?" H 4000 4250 40  0000 L CNN
+F 0 "C10" H 4000 4250 40  0000 L CNN
 F 1 "1U" H 4006 4065 40  0000 L CNN
 F 2 "~" H 4038 4000 30  0000 C CNN
@@
 $EndComp
 $Comp
-L R R?
+L R R17
 U 1 1 5302A340
 P 4950 4800
-F 0 "R?" V 5030 4800 40  0000 C CNN
+F 0 "R17" V 5030 4800 40  0000 C CNN
 F 1 "10K" V 4957 4801 40  0000 C CNN
 F 2 "~" V 4880 4800 30  0000 C CNN
@@
 $EndComp
 $Comp
-L GND #PWR?
+L GND #PWR022
 U 1 1 5302A369
 P 4000 5150
-F 0 "#PWR?" H 4000 5150 30  0001 C CNN
+F 0 "#PWR022" H 4000 5150 30  0001 C CNN
 F 1 "GND" H 4000 5080 30  0001 C CNN
 F 2 "" H 4000 5150 60  0000 C CNN
@@
 $EndComp
 $Comp
-L R R?
+L R R16
 U 1 1 5302A38C
 P 4850 4350
-F 0 "R?" V 4930 4350 40  0000 C CNN
+F 0 "R16" V 4930 4350 40  0000 C CNN
 F 1 "R" V 4857 4351 40  0000 C CNN
 F 2 "~" V 4780 4350 30  0000 C CNN
@@
 Connection ~ 4450 5050
 $Comp
-L R R?
+L R R15
 U 1 1 5302A3F3
 P 4850 4050
-F 0 "R?" V 4930 4050 40  0000 C CNN
+F 0 "R15" V 4930 4050 40  0000 C CNN
 F 1 "1,6K" V 4857 4051 40  0000 C CNN
 F 2 "~" V 4780 4050 30  0000 C CNN
@@
 Connection ~ 4450 4200
 $Comp
-L R R?
+L R R18
 U 1 1 5302A43C
 P 6800 4700
-F 0 "R?" V 6880 4700 40  0000 C CNN
+F 0 "R18" V 6880 4700 40  0000 C CNN
 F 1 "R" V 6807 4701 40  0000 C CNN
 F 2 "~" V 6730 4700 30  0000 C CNN
@@
 en
 $Comp
-L LED D?
+L LED D4
 U 1 1 5302A4A4
 P 7200 4200
-F 0 "D?" H 7200 4300 50  0000 C CNN
+F 0 "D4" H 7200 4300 50  0000 C CNN
 F 1 "LED_YELLOW" H 7200 4100 50  0000 C CNN
 F 2 "~" H 7200 4200 60  0000 C CNN
@@
 Connection ~ 6900 4200
 $Comp
-L R R?
+L R R19
 U 1 1 5302A4EB
 P 7550 3800
-F 0 "R?" V 7630 3800 40  0000 C CNN
+F 0 "R19" V 7630 3800 40  0000 C CNN
 F 1 "1K" V 7557 3801 40  0000 C CNN
 F 2 "~" V 7480 3800 30  0000 C CNN
@@
 PACK+
 $Comp
-L +3.3V #PWR?
+L +3.3V #PWR023
 U 1 1 5302A53C
 P 7550 3400
-F 0 "#PWR?" H 7550 3360 30  0001 C CNN
+F 0 "#PWR023" H 7550 3360 30  0001 C CNN
 F 1 "+3.3V" H 7550 3510 30  0000 C CNN
 F 2 "" H 7550 3400 60  0000 C CNN
