File: PUA-201410/cohete_2014/cohete.sch (KiCad schematic (older format))
At the start: 30 parts, among them IC1 ATXMEGA32A4U-A, M1 XBEE-PRO, P1 CONN_2, P2 CONN_4, P3 CONN_6, P4 CONN_4, P5 CONN_8, U1 LM1117, U2 L78S05, X1 CRYSTAL

Commit message: corrección PUA
con resistencias de pulldown y archivos de fabricación
Parts:
- removed P2: CONN_4, symbol CONN_4
- added P2: CONN_6, symbol CONN_6
- added R10, R11, R12, R8, R9: 1K, ~, symbol R
- C1, C2: value C -> 22pF
- R1, R2: value R -> 4.7K
- R3: value 1K -> 2K
- R4, R5, R7: value R -> 1K
- R6: value 500 -> 1k
- X1: value CRYSTAL -> 32Mhz
Connections:
- net GND: now also P2.1, R10.2, R11.2, R12.2, R8.2, R9.2
- net IGN_0: now also P2.2, R8.1
- net IGN_1: now also P2.3, R9.1
- net IGN_2: now also P2.4, R10.1
- net IGN_3: now reaches IC1.23 (PD3)
- net IGN_3: now also P2.5, R11.1
- net EN_IGN: now reaches IC1.24 (PD4)
- net EN_IGN: now also P2.6, R12.1
